File: rov_esc/rov_esc.kicad_pcb (KiCad board)
At the start: 2 copper layers, 35 parts

Commit message: Update UnderWater-Rov-KOU-GALLIPOLI.iml
Parts:
- removed the ? at (362.1, 165.8)
- removed the ? at (350.0, 23.6)
- removed the ? at (291.0, 25.3)
- removed the ? at (116.2, 168.9)
- removed the ? at (116.6, 116.0)
- removed the ? at (245.6, 45.7)
- removed the REF** at (131.1, 154.3)
- removed the REF** at (113.6, 50.7)
- removed the REF** at (144.7, 32.7)
- removed the REF** at (132.1, 100.9)
- removed the REF** at (120.7, 100.9)
- removed the REF** at (344.7, 166.0)
- removed the REF** at (352.0, 163.9)
- removed the REF** at (348.1, 33.7)
- removed the REF** at (350.2, 41.1)
- removed the REF** at (289.1, 35.4)
- removed the REF** at (291.2, 42.7)
- removed the REF** at (346.8, 180.2)
- removed the REF** at (133.7, 168.7)
- removed the REF** at (126.3, 170.8)
- removed the REF** at (126.7, 117.9)
- removed the REF** at (134.0, 115.8)
- removed the REF** at (129.0, 32.4)
- removed the REF** at (243.6, 55.8)
- removed the REF** at (245.8, 63.1)
- removed the REF** at (119.2, 154.5)
- removed the REF** at (359.9, 180.4)
- removed the REF** at (305.8, 40.7)
- removed the REF** at (364.7, 38.3)
- removed the REF** at (364.8, 25.3)
- removed the REF** at (305.6, 26.8)
- removed the REF** at (248.9, 37.0)
- removed Sinyal: ESC0 Giriş, Connector_PinHeader_2.00mm:PinHeader_1x03_P2.00mm_Vertical
- removed Sinyal: PinHeader_1x03_P2.00mm_Vertical, Connector_PinHeader_2.00mm:PinHeader_1x03_P2.00mm_Vertical
- added REF**: AMASS_XT60-F_1x02_P7.20mm_Vertical, Connector_AMASS:AMASS_XT60-F_1x02_P7.20mm_Vertical, F.Cu at (341.7, 106.3)
- added REF**: PinHeader_1x12_P2.54mm_Vertical, Connector_PinHeader_2.54mm:PinHeader_1x12_P2.54mm_Vertical, F.Cu at (387.6, 92.8)
- added REF**: PinHeader_2x02_P2.54mm_Vertical, Connector_PinHeader_2.54mm:PinHeader_2x02_P2.54mm_Vertical, F.Cu at (426.2, 72.8)
- added REF**: PinHeader_2x02_P2.54mm_Vertical, Connector_PinHeader_2.54mm:PinHeader_2x02_P2.54mm_Vertical, F.Cu at (426.0, 46.0)
- added REF**: PinHeader_1x08_P2.54mm_Vertical, Connector_PinHeader_2.54mm:PinHeader_1x08_P2.54mm_Vertical, F.Cu at (397.8, 103.7)
- added REF**: AMASS_XT60-F_1x02_P7.20mm_Vertical, Connector_AMASS:AMASS_XT60-F_1x02_P7.20mm_Vertical, F.Cu at (368.5, 94.0)
- added REF**: PinHeader_1x12_P2.54mm_Vertical, Connector_PinHeader_2.54mm:PinHeader_1x12_P2.54mm_Vertical, F.Cu at (387.8, 97.1)
- added REF**: PinHeader_1x08_P2.54mm_Vertical, Connector_PinHeader_2.54mm:PinHeader_1x08_P2.54mm_Vertical, F.Cu at (397.8, 108.6)
- added REF**: PinHeader_1x12_P2.54mm_Vertical, Connector_PinHeader_2.54mm:PinHeader_1x12_P2.54mm_Vertical, F.Cu at (387.7, 103.6)
- added REF**: PinHeader_1x12_P2.54mm_Vertical, Connector_PinHeader_2.54mm:PinHeader_1x12_P2.54mm_Vertical, F.Cu at (387.8, 108.6)
- added REF**: PinHeader_1x12_P2.54mm_Vertical, Connector_PinHeader_2.54mm:PinHeader_1x12_P2.54mm_Vertical, F.Cu at (240.0, 107.6)
- added REF**: AMASS_XT60-F_1x02_P7.20mm_Vertical, Connector_AMASS:AMASS_XT60-F_1x02_P7.20mm_Vertical, F.Cu at (320.0, 106.5)
- added REF**: PinHeader_1x12_P2.54mm_Vertical, Connector_PinHeader_2.54mm:PinHeader_1x12_P2.54mm_Vertical, F.Cu at (239.9, 102.6)
- added REF**: PinHeader_1x08_P2.54mm_Vertical, Connector_PinHeader_2.54mm:PinHeader_1x08_P2.54mm_Vertical, F.Cu at (250.0, 107.6)
- added REF**: PinHeader_1x08_P2.54mm_Vertical, Connector_PinHeader_2.54mm:PinHeader_1x08_P2.54mm_Vertical, F.Cu at (250.0, 102.7)
- added REF**: PinHeader_2x02_P2.54mm_Vertical, Connector_PinHeader_2.54mm:PinHeader_2x02_P2.54mm_Vertical, F.Cu at (278.2, 45.0)
- added REF**: PinHeader_2x02_P2.54mm_Vertical, Connector_PinHeader_2.54mm:PinHeader_2x02_P2.54mm_Vertical, F.Cu at (278.5, 71.8)
- added REF**: PinHeader_1x12_P2.54mm_Vertical, Connector_PinHeader_2.54mm:PinHeader_1x12_P2.54mm_Vertical, F.Cu at (239.8, 91.8)
- added REF**: PinHeader_1x12_P2.54mm_Vertical, Connector_PinHeader_2.54mm:PinHeader_1x12_P2.54mm_Vertical, F.Cu at (240.0, 96.1)
- added REF**: AMASS_XT60-F_1x02_P7.20mm_Vertical, Connector_AMASS:AMASS_XT60-F_1x02_P7.20mm_Vertical, F.Cu at (220.7, 105.4)
- added REF**: AMASS_XT60-F_1x02_P7.20mm_Vertical, Connector_AMASS:AMASS_XT60-F_1x02_P7.20mm_Vertical, F.Cu at (220.7, 93.0)
- added REF**: AMASS_XT60-F_1x02_P7.20mm_Vertical, Connector_AMASS:AMASS_XT60-F_1x02_P7.20mm_Vertical, F.Cu at (171.6, 27.7)
- added REF**: AMASS_XT60-F_1x02_P7.20mm_Vertical, Connector_AMASS:AMASS_XT60-F_1x02_P7.20mm_Vertical, F.Cu at (319.2, 42.1)
- added REF**: AMASS_XT60-F_1x02_P7.20mm_Vertical, Connector_AMASS:AMASS_XT60-F_1x02_P7.20mm_Vertical, F.Cu at (192.9, 27.9)
- added REF**: AMASS_XT60-F_1x02_P7.20mm_Vertical, Connector_AMASS:AMASS_XT60-F_1x02_P7.20mm_Vertical, F.Cu at (193.1, 41.1)
- added REF**: AMASS_XT60-F_1x02_P7.20mm_Vertical, Connector_AMASS:AMASS_XT60-F_1x02_P7.20mm_Vertical, F.Cu at (171.4, 41.1)
- added REF**: AMASS_XT60-F_1x02_P7.20mm_Vertical, Connector_AMASS:AMASS_XT60-F_1x02_P7.20mm_Vertical, F.Cu at (172.2, 92.5)
- added REF**: AMASS_XT60-F_1x02_P7.20mm_Vertical, Connector_AMASS:AMASS_XT60-F_1x02_P7.20mm_Vertical, F.Cu at (193.9, 92.9)
- added REF**: AMASS_XT60-F_1x02_P7.20mm_Vertical, Connector_AMASS:AMASS_XT60-F_1x02_P7.20mm_Vertical, F.Cu at (193.9, 105.3)
- added REF**: AMASS_XT60-F_1x02_P7.20mm_Vertical, Connector_AMASS:AMASS_XT60-F_1x02_P7.20mm_Vertical, F.Cu at (172.2, 105.5)
- added REF**: AMASS_XT60-F_1x02_P7.20mm_Vertical, Connector_AMASS:AMASS_XT60-F_1x02_P7.20mm_Vertical, F.Cu at (320.0, 93.5)
- added REF**: AMASS_XT60-F_1x02_P7.20mm_Vertical, Connector_AMASS:AMASS_XT60-F_1x02_P7.20mm_Vertical, F.Cu at (341.7, 93.9)
- added REF**: AMASS_XT60-F_1x02_P7.20mm_Vertical, Connector_AMASS:AMASS_XT60-F_1x02_P7.20mm_Vertical, F.Cu at (340.9, 42.1)
- added REF**: AMASS_XT60-F_1x02_P7.20mm_Vertical, Connector_AMASS:AMASS_XT60-F_1x02_P7.20mm_Vertical, F.Cu at (340.7, 28.9)
- added REF**: AMASS_XT60-F_1x02_P7.20mm_Vertical, Connector_AMASS:AMASS_XT60-F_1x02_P7.20mm_Vertical, F.Cu at (319.4, 28.7)
- added REF**: AMASS_XT60-F_1x02_P7.20mm_Vertical, Connector_AMASS:AMASS_XT60-F_1x02_P7.20mm_Vertical, F.Cu at (368.5, 106.3)
Routing:
- net (no net): track 1158.5 -> 1535.4 mm, vias 54 -> 4
Other:
- net class Default: trace_width 3 -> 6
- board text added: "12v"
- board text added: "5v"
- board text added: "GND"
- board text removed: "+12v"
- board text removed: "-12v"
- board text removed: "DownLeft ESC1"
- board text removed: "DownRight ESC0"
- board text removed: "ESC0"
- board text removed: "ESC1"
- board text removed: "Sinyal"
