File: rov_pcb/rov_pcb.kicad_pcb (KiCad board)
At the start: 2 copper layers, 10 parts

Commit message: Update UnderWater-Rov-KOU-GALLIPOLI.iml
Parts:
- removed the REF** at (128.1, 46.8)
- removed the REF** at (128.0, 65.9)
- removed the REF** at (148.2, 46.2)
- removed the REF** at (145.5, 46.2)
- removed the REF** at (142.5, 46.2)
- removed the REF** at (74.3, 64.5)
- removed the REF** at (76.9, 64.6)
- removed the REF** at (88.4, 65.6)
- removed the REF** at (88.5, 47.0)
- removed the RP? at (127.0, 126.2)
- added REF**: PinHeader_1x02_P2.54mm_Vertical, Connector_PinHeader_2.54mm:PinHeader_1x02_P2.54mm_Vertical, F.Cu at (343.3, 168.3)
- added REF**: PinHeader_1x02_P2.54mm_Horizontal, Connector_PinHeader_2.54mm:PinHeader_1x02_P2.54mm_Horizontal, F.Cu at (297.1, 122.3)
- added REF**: PinHeader_1x02_P2.54mm_Horizontal, Connector_PinHeader_2.54mm:PinHeader_1x02_P2.54mm_Horizontal, F.Cu at (304.3, 122.2)
- added REF**: PinHeader_1x02_P2.54mm_Horizontal, Connector_PinHeader_2.54mm:PinHeader_1x02_P2.54mm_Horizontal, F.Cu at (309.7, 122.2)
- added REF**: PinHeader_1x02_P2.54mm_Horizontal, Connector_PinHeader_2.54mm:PinHeader_1x02_P2.54mm_Horizontal, F.Cu at (331.1, 145.5)
- added REF**: PinHeader_1x02_P2.54mm_Horizontal, Connector_PinHeader_2.54mm:PinHeader_1x02_P2.54mm_Horizontal, F.Cu at (342.8, 177.5)
- added REF**: PinHeader_1x02_P2.54mm_Vertical, Connector_PinHeader_2.54mm:PinHeader_1x02_P2.54mm_Vertical, F.Cu at (343.1, 163.9)
- added REF**: PinHeader_1x02_P2.54mm_Vertical, Connector_PinHeader_2.54mm:PinHeader_1x02_P2.54mm_Vertical, F.Cu at (343.3, 172.3)
- added REF**: PinHeader_1x02_P2.54mm_Horizontal, Connector_PinHeader_2.54mm:PinHeader_1x02_P2.54mm_Horizontal, F.Cu at (330.9, 174.8)
- added REF**: PinHeader_1x02_P2.54mm_Vertical, Connector_PinHeader_2.54mm:PinHeader_1x02_P2.54mm_Vertical, F.Cu at (343.0, 180.7)
- added REF**: PinHeader_1x08_P2.54mm_Vertical, Connector_PinHeader_2.54mm:PinHeader_1x08_P2.54mm_Vertical, F.Cu at (335.8, 164.5)
- added REF**: PinHeader_1x12_P2.54mm_Horizontal, Connector_PinHeader_2.54mm:PinHeader_1x12_P2.54mm_Horizontal, F.Cu at (265.5, 122.0)
- added REF**: PinHeader_1x15_P2.54mm_Horizontal, Connector_PinHeader_2.54mm:PinHeader_1x15_P2.54mm_Horizontal, F.Cu at (260.2, 153.9)
- added REF**: PinHeader_1x02_P2.54mm_Vertical, Connector_PinHeader_2.54mm:PinHeader_1x02_P2.54mm_Vertical, F.Cu at (343.1, 160.1)
- added REF**: PinHeader_1x02_P2.54mm_Vertical, Connector_PinHeader_2.54mm:PinHeader_1x02_P2.54mm_Vertical, F.Cu at (343.1, 152.4)
- added REF**: PinHeader_1x08_P2.54mm_Vertical, Connector_PinHeader_2.54mm:PinHeader_1x08_P2.54mm_Vertical, F.Cu at (335.9, 135.5)
- added REF**: PinHeader_1x02_P2.54mm_Vertical, Connector_PinHeader_2.54mm:PinHeader_1x02_P2.54mm_Vertical, F.Cu at (343.1, 156.2)
- added REF**: PinHeader_1x15_P2.54mm_Horizontal, Connector_PinHeader_2.54mm:PinHeader_1x15_P2.54mm_Horizontal, F.Cu at (295.8, 178.6)
- added REF**: PinHeader_1x15_P2.54mm_Horizontal, Connector_PinHeader_2.54mm:PinHeader_1x15_P2.54mm_Horizontal, F.Cu at (295.8, 141.8)
- added REF**: PinHeader_1x18_P2.54mm_Vertical, Connector_PinHeader_2.54mm:PinHeader_1x18_P2.54mm_Vertical, F.Cu at (262.8, 130.5)
- added REF**: PinHeader_1x02_P2.54mm_Horizontal, Connector_PinHeader_2.54mm:PinHeader_1x02_P2.54mm_Horizontal, F.Cu at (192.8, 177.5)
- added REF**: PinHeader_1x02_P2.54mm_Horizontal, Connector_PinHeader_2.54mm:PinHeader_1x02_P2.54mm_Horizontal, F.Cu at (192.9, 148.0)
- added REF**: PinHeader_1x08_P2.54mm_Horizontal, Connector_PinHeader_2.54mm:PinHeader_1x08_P2.54mm_Horizontal, F.Cu at (304.5, 81.1)
- added REF**: PinHeader_1x02_P2.54mm_Horizontal, Connector_PinHeader_2.54mm:PinHeader_1x02_P2.54mm_Horizontal, F.Cu at (181.1, 145.5)
- added REF**: PinHeader_1x02_P2.54mm_Horizontal, Connector_PinHeader_2.54mm:PinHeader_1x02_P2.54mm_Horizontal, F.Cu at (165.7, 174.7)
- added REF**: PinHeader_1x02_P2.54mm_Horizontal, Connector_PinHeader_2.54mm:PinHeader_1x02_P2.54mm_Horizontal, F.Cu at (180.9, 174.8)
- added REF**: PinHeader_1x02_P2.54mm_Horizontal, Connector_PinHeader_2.54mm:PinHeader_1x02_P2.54mm_Horizontal, F.Cu at (177.3, 177.4)
- added REF**: PinHeader_1x08_P2.54mm_Horizontal, Connector_PinHeader_2.54mm:PinHeader_1x08_P2.54mm_Horizontal, F.Cu at (175.4, 102.9)
- added REF**: PinHeader_1x08_P2.54mm_Horizontal, Connector_PinHeader_2.54mm:PinHeader_1x08_P2.54mm_Horizontal, F.Cu at (154.5, 81.1)
- added REF**: PinHeader_1x02_P2.54mm_Horizontal, Connector_PinHeader_2.54mm:PinHeader_1x02_P2.54mm_Horizontal, F.Cu at (164.8, 122.2)
- added REF**: PinHeader_1x02_P2.54mm_Horizontal, Connector_PinHeader_2.54mm:PinHeader_1x02_P2.54mm_Horizontal, F.Cu at (159.7, 122.2)
- added REF**: PinHeader_1x02_P2.54mm_Horizontal, Connector_PinHeader_2.54mm:PinHeader_1x02_P2.54mm_Horizontal, F.Cu at (154.3, 122.2)
- added REF**: PinHeader_1x02_P2.54mm_Horizontal, Connector_PinHeader_2.54mm:PinHeader_1x02_P2.54mm_Horizontal, F.Cu at (147.1, 122.3)
- added REF**: PinHeader_1x02_P2.54mm_Horizontal, Connector_PinHeader_2.54mm:PinHeader_1x02_P2.54mm_Horizontal, F.Cu at (314.8, 122.2)
- added REF**: PinHeader_1x12_P2.54mm_Horizontal, Connector_PinHeader_2.54mm:PinHeader_1x12_P2.54mm_Horizontal, F.Cu at (115.5, 122.0)
- added REF**: PinHeader_1x17_P2.54mm_Vertical, Connector_PinHeader_2.54mm:PinHeader_1x17_P2.54mm_Vertical, F.Cu at (190.3, 82.1)
- added REF**: PinHeader_1x02_P2.54mm_Vertical, Connector_PinHeader_2.54mm:PinHeader_1x02_P2.54mm_Vertical, F.Cu at (193.0, 180.7)
- added REF**: PinHeader_1x02_P2.54mm_Vertical, Connector_PinHeader_2.54mm:PinHeader_1x02_P2.54mm_Vertical, F.Cu at (193.3, 172.3)
- added REF**: PinHeader_1x02_P2.54mm_Vertical, Connector_PinHeader_2.54mm:PinHeader_1x02_P2.54mm_Vertical, F.Cu at (193.3, 168.3)
- added REF**: PinHeader_1x02_P2.54mm_Vertical, Connector_PinHeader_2.54mm:PinHeader_1x02_P2.54mm_Vertical, F.Cu at (193.1, 163.9)
- added REF**: PinHeader_1x02_P2.54mm_Vertical, Connector_PinHeader_2.54mm:PinHeader_1x02_P2.54mm_Vertical, F.Cu at (193.1, 160.1)
- added REF**: PinHeader_1x02_P2.54mm_Vertical, Connector_PinHeader_2.54mm:PinHeader_1x02_P2.54mm_Vertical, F.Cu at (193.1, 156.2)
- added REF**: PinHeader_1x02_P2.54mm_Vertical, Connector_PinHeader_2.54mm:PinHeader_1x02_P2.54mm_Vertical, F.Cu at (193.1, 152.4)
- added REF**: PinHeader_1x15_P2.54mm_Horizontal, Connector_PinHeader_2.54mm:PinHeader_1x15_P2.54mm_Horizontal, F.Cu at (145.8, 178.6)
- added REF**: PinHeader_1x08_P2.54mm_Horizontal, Connector_PinHeader_2.54mm:PinHeader_1x08_P2.54mm_Horizontal, F.Cu at (325.4, 102.9)
- added REF**: PinHeader_1x15_P2.54mm_Horizontal, Connector_PinHeader_2.54mm:PinHeader_1x15_P2.54mm_Horizontal, F.Cu at (110.2, 153.9)
- added REF**: PinHeader_1x15_P2.54mm_Horizontal, Connector_PinHeader_2.54mm:PinHeader_1x15_P2.54mm_Horizontal, F.Cu at (145.8, 141.8)
- added REF**: PinHeader_1x18_P2.54mm_Vertical, Connector_PinHeader_2.54mm:PinHeader_1x18_P2.54mm_Vertical, F.Cu at (112.8, 130.5)
- added REF**: PinHeader_1x08_P2.54mm_Vertical, Connector_PinHeader_2.54mm:PinHeader_1x08_P2.54mm_Vertical, F.Cu at (185.8, 164.5)
- added REF**: PinHeader_1x08_P2.54mm_Vertical, Connector_PinHeader_2.54mm:PinHeader_1x08_P2.54mm_Vertical, F.Cu at (185.9, 135.5)
- added REF**: PinHeader_1x02_P2.54mm_Horizontal, Connector_PinHeader_2.54mm:PinHeader_1x02_P2.54mm_Horizontal, F.Cu at (315.7, 174.7)
- added REF**: PinHeader_1x02_P2.54mm_Horizontal, Connector_PinHeader_2.54mm:PinHeader_1x02_P2.54mm_Horizontal, F.Cu at (327.3, 177.4)
- added REF**: PinHeader_1x17_P2.54mm_Vertical, Connector_PinHeader_2.54mm:PinHeader_1x17_P2.54mm_Vertical, F.Cu at (340.3, 82.1)
- added REF**: PinHeader_1x02_P2.54mm_Horizontal, Connector_PinHeader_2.54mm:PinHeader_1x02_P2.54mm_Horizontal, F.Cu at (342.9, 148.0)
- added RP?: Raspberry_Pi_2_3, Raspberry-Pi-3-library-for-kicad-master:rasberry, B.Cu at (284.4, 136.4)
- added RP?: Raspberry_Pi_2_3, Raspberry-Pi-3-library-for-kicad-master:rasberry, B.Cu at (134.4, 136.4)
- added XA**: Arduino_Mega2560_Shield, Arduino:Arduino_Mega2560_Shield, B.Cu at (235.8, 74.7)
- added XA**: Arduino_Mega2560_Shield, Arduino:Arduino_Mega2560_Shield, B.Cu at (85.8, 74.7)
Routing:
- net (no net): track 240.1 -> 3967.6 mm, vias 6 -> 2
- added copper zone on B.Cu, net (none)
Other:
- net class Default: via_dia 0.8 -> 2; via_drill 0.4 -> 1
- board text added: "ANALOG PİNS 0-7"
- board text added: "DİGİTAL PWM PİNS 2-13"
- board text added: "DİGİTAL PİNS 38-52"
- board text added: "GND"
- board text added: "MEGA DİGİTAL PİNS 23-53"
- board text added: "MEGA I2C"
- board text added: "ORTADAN PİNLERİN DURUMUNA GÖRE KESİLEBİLİR"
- board text added: "RP I2C"
- board text added: "RX TX"
- board text added: "SCL"
- board text added: "SDA"
- board text added: "UART PİNS 1-3"
